Commit message: Move robot model to ROS package

File: ros/ieee2015_robot/urdf/IEEEurdf.URDF (robot description, URDF)
Before this commit: robot robot, 8 links, 7 joints
Links:
- added link camera_link, mass 1e-5; collision box size=0.025 0.025 0.025; visual box size=0.025 0.025 0.025
- link ArmRot1: geometry collision mesh filename=package://ieee2015_robot/meshes/ArmRot1_col.STL; visual mesh filename=package://ieee2015_robot/meshes/ArmRot1.STL
- link ArmRot2: geometry collision mesh filename=package://ieee2015_robot/meshes/ArmRot2_col.STL; visual mesh filename=package://ieee2015_robot/meshes/ArmRot2.STL
- link ArmYRot: geometry collision mesh filename=package://ieee2015_robot/meshes/ArmYRot_col.STL; visual mesh filename=package://ieee2015_robot/meshes/ArmYRot.STL
- link BLWheel: geometry collision mesh filename=package://ieee2015_robot/meshes/BLWheel_col.STL; visual mesh filename=package://ieee2015_robot/meshes/BLWheel.STL
- link BRWheel: geometry collision mesh filename=package://ieee2015_robot/meshes/BRWheel_col.STL; visual mesh filename=package://ieee2015_robot/meshes/BRWheel.STL
- link FLWheel: geometry collision mesh filename=package://ieee2015_robot/meshes/FLWheel_col.STL; visual mesh filename=package://ieee2015_robot/meshes/FLWheel.STL
- link FRWheel: geometry collision mesh filename=package://ieee2015_robot/meshes/FRWheel_col.STL; visual mesh filename=package://ieee2015_robot/meshes/FRWheel.STL
- link base_link: geometry collision mesh filename=package://ieee2015_robot/meshes/base_link_col.STL; visual mesh filename=package://ieee2015_robot/meshes/base_link.STL
Joints:
- added joint camera_joint: type fixed, parent base_link, child camera_link, origin xyz=0 -.15 .040 rpy=0 0 -1.57, axis 1 0 0

Commit message: Added arm control using ros_control

File: ros/ieee2015_robot/urdf/IEEEurdf.URDF (robot description, URDF)
Before this commit: robot ieee2015_robot, 9 links, 8 joints
Links:
- added link kinect_link, mass 1e-5; collision box size=0.1 0.025 0.025; visual box size=0.025 0.1 0.025
- link ArmRot1: mass 0.247629627425225 -> 0.187629627425225
- link ArmRot2: mass 0.274282093236145 -> 0.204282093236145
- link ArmYRot: mass 0.571743531126574 -> 0.271743531126574
- link base_link: mass 1.15919256315212 -> 15.15919256315212
Joints:
- added joint kinect_joint: type fixed, parent base_link, child kinect_link, origin xyz=0 -.1 .04 rpy=0 0 -1.57, axis 1 0 0
- joint ArmRot1Rev: limit lower=0 upper=0 effort=10 velocity=1 -> lower=-1.77 upper=1.37 effort=10 velocity=1
- joint ArmRot2Rev: limit lower=0 upper=0 effort=10 velocity=1 -> lower=-5 upper=.9 effort=10 velocity=1
- joint ArmYRotCont: limit (none) -> lower=-999 upper=999 effort=10 velocity=1; origin xyz=0 0 0.02266 rpy=1.5708 -4.2993E-16 -0.7854 -> xyz=0 0 0.02266 rpy=1.5708 -4.2993E-16 -3.14; type continuous -> revolute
- joint camera_joint: origin xyz=0 -.15 .040 rpy=0 0 -1.57 -> xyz=0 -.15 -.015 rpy=0 0 -1.57

Commit message: Updated arm control

File: ros/ieee2015_robot/urdf/IEEEurdf.URDF (robot description, URDF)
Before this commit: robot ieee2015_robot, 10 links, 9 joints
Links:
- link ArmRot1: geometry visual mesh filename=package://ieee2015_robot/meshes/ArmRot1.STL
- link ArmRot2: geometry visual mesh filename=package://ieee2015_robot/meshes/ArmRot2.STL
Joints:
- joint ArmRot1Rev: limit lower=-1.77 upper=1.37 effort=10 velocity=1 -> lower=-3.14 upper=3.14 effort=10 velocity=1; origin xyz=1.143E-05 0.057267 0.020728 rpy=-7.3956E-32 -1.1102E-16 1.7931E-21 -> xyz=1.143E-05 0.057267 0.020728 rpy=1.35 -1.1102E-16 1.7931E-21
- joint ArmRot2Rev: limit lower=-5 upper=.9 effort=10 velocity=1 -> lower=-3 upper=3 effort=10 velocity=1; origin xyz=-1.143E-05 0.13289 0.065139 rpy=4.9304E-32 0 6.1824E-18 -> xyz=-1.143E-05 0.13289 0.065139 rpy=-2.1 0 6.1824E-18

Commit message: Git is telling me to push this, ignore

File: ros/ieee2015_robot/urdf/IEEEurdf.URDF (robot description, URDF)
Before this commit: robot ieee2015_robot, 10 links, 9 joints
Joints:
- joint camera_joint: origin xyz=0 -.15 -.015 rpy=0 0 -1.57 -> xyz=0 -.15 .020 rpy=0 .587 -1.57
